File: RS232-Shield/RS232-shield.sch (KiCad schematic (older format))
At the start: 12 parts, among them J1 DB9_Female_MountingHoles, U1 WeMos_D1_mini, U2 MAX3232

Commit message: Add RS-232 Shield PCB layout
Parts:
- U1: symbol MCU_Module:WeMos_D1_mini -> shieldLibrary:WeMos_D1_mini
Changed lines of the file:
@@
 NoConn ~ 7950 4200
 $Comp
-L MCU_Module:WeMos_D1_mini U1
+L shieldLibrary:WeMos_D1_mini U1
 U 1 1 60CF9E07
 P 1600 3950

Commit message: Modify PCB silkscreens
Project-specific footprint added for Wemos D1 Mini
Parts:
- U1: footprint Module:WEMOS_D1_mini_light -> RS232-shield:WEMOS_D1_mini_light
Changed lines of the file:
@@
 F 0 "U1" H 1350 3150 50  0000 C CNN
 F 1 "WeMos_D1_mini" V 1250 3550 50  0000 C CNN
-F 2 "Module:WEMOS_D1_mini_light" H 1600 2800 50  0001 C CNN
+F 2 "RS232-shield:WEMOS_D1_mini_light" H 1600 2800 50  0001 C CNN
 F 3 "https://wiki.wemos.cc/products:d1:d1_mini#documentation" H -250 2800 50  0001 C CNN
 	1    1600 3950
